File: hardware/dennisquad.brd (EAGLE design)
At the start: 25 x 25 mm, 45 parts, among them Q1 FA-128, U1 MCP1700T-3302E/MAY, U2 NRF52832_QFN48, U3 DRV8839, U4 DRV8839, U5 MPU-9250, U6 LPS25HB, X1 CRYSTAL.ABS07

Commit message: Minor changes
Routing:
- net GND: vias 66 -> 71
Changed lines of the file:
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@@
 </element>
 <element name="C9" library="SparkFun-Capacitors" package="0402-CAP" value="100pF" x="11.425" y="13.225" smashed="yes" rot="R180">
-<attribute name="NAME" x="10.186" y="13.8735" size="0.4064" layer="25"/>
+<attribute name="NAME" x="10.286" y="13.8985" size="0.4064" layer="25"/>
 <attribute name="MPN" value="GRM1555C1H101JA01D" x="11.425" y="13.225" size="1.778" layer="27" rot="R180" display="off"/>
 </element>
@@
 <attribute name="MPN" value="GRM1555C1H160GA01D" x="11.5" y="8.575" size="1.778" layer="27" rot="R180" display="off"/>
 </element>
-<element name="C8" library="SparkFun-Capacitors" package="0402-CAP" value="16pF" x="9.875" y="10.59" smashed="yes" rot="R90">
-<attribute name="NAME" x="9.186" y="11.8385" size="0.4064" layer="25"/>
-<attribute name="MPN" value="GRM1555C1H160GA01D" x="9.875" y="10.59" size="1.778" layer="27" rot="R90" display="off"/>
+<element name="C8" library="SparkFun-Capacitors" package="0402-CAP" value="16pF" x="9.9" y="10.59" smashed="yes" rot="R90">
+<attribute name="NAME" x="9.511" y="11.8385" size="0.4064" layer="25"/>
+<attribute name="MPN" value="GRM1555C1H160GA01D" x="9.9" y="10.59" size="1.778" layer="27" rot="R90" display="off"/>
 </element>
 <element name="RESET" library="omron" package="B3U-1000P(M)" value="SPST.B3U-1000P(M)" x="7.25" y="22.55" smashed="yes" rot="R90">
@@
 <attribute name="VALUE" x="7.045" y="11.82" size="1.27" layer="27" rot="R90"/>
 </element>
-<element name="U$1" library="SparkFun-RF" package="ANTENNA-W3008C" value="ANTENNA-W3008C" x="6.9" y="11.85"/>
+<element name="U$1" library="SparkFun-RF" package="ANTENNA-W3008C" value="ANTENNA-W3008C" x="6.9" y="11.85">
+<attribute name="MPN" value="W3008C" x="6.9" y="11.85" size="0.5" layer="27" display="off"/>
+</element>
 </elements>
 <signals>
@@
 <contactref element="U1" pad="P$1"/>
 <contactref element="CN1" pad="2"/>
-<via x="4.575" y="11.525" extent="1-16" drill="0.254"/>
-<via x="4.575" y="11.025" extent="1-16" drill="0.254"/>
-<via x="4.575" y="10.525" extent="1-16" drill="0.254"/>
-<via x="4.575" y="10.025" extent="1-16" drill="0.254"/>
-<via x="4.575" y="9.525" extent="1-16" drill="0.254"/>
+<via x="4.575" y="11.425" extent="1-16" drill="0.254"/>
+<via x="4.575" y="10.925" extent="1-16" drill="0.254"/>
+<via x="4.575" y="10.425" extent="1-16" drill="0.254"/>
+<via x="4.575" y="9.925" extent="1-16" drill="0.254"/>
+<via x="4.575" y="9.425" extent="1-16" drill="0.254"/>
 <via x="11.325" y="3.125" extent="1-16" drill="0.254"/>
 <via x="5.075" y="4.675" extent="1-16" drill="0.254"/>
@@
 <via x="0.675" y="19.475" extent="1-16" drill="0.254"/>
 <via x="2.725" y="12.225" extent="1-16" drill="0.254"/>
+<via x="9.05" y="9.45" extent="1-16" drill="0.254"/>
+<via x="4.55" y="8.925" extent="1-16" drill="0.254"/>
+<via x="4.575" y="11.925" extent="1-16" drill="0.254"/>
+<via x="9.15" y="12.35" extent="1-16" drill="0.254"/>
+<via x="9.15" y="11.85" extent="1-16" drill="0.254"/>
 </signal>
 <signal name="VCC">
@@
 <wire x1="13.55" y1="13.75" x2="12.9" y2="13.75" width="0.127" layer="16"/>
 <wire x1="12.9" y1="13.75" x2="11.35" y2="12.2" width="0.127" layer="16"/>
-<wire x1="9.875" y1="11.17" x2="10.23" y2="11.325" width="0.127" layer="1"/>
+<wire x1="9.9" y1="11.17" x2="10.23" y2="11.325" width="0.127" layer="1"/>
 <wire x1="10.23" y1="11.325" x2="11.15" y2="11.325" width="0.127" layer="1"/>
 </signal>

Commit message: Minor fixes
Parts:
- U1: value MCP1700T-3302E/MAY -> NRF52832_QFN48; device wrea:6-VDFN -> nRF52Series:QFN48
- U2: value NRF52832_QFN48 -> MCP1700T-3302E/MAY; device nRF52Series:QFN48 -> wrea:6-VDFN
- moved U1 15.9 mm to (17.8, 15.5), turned to 90 degrees
- moved U2 15.9 mm to (7.30, 3.52), turned to 180 degrees
- moved C12 0.10 mm to (9.88, 2.45)
- moved C6 0.10 mm to (9.90, 4.03)
- renumbered U$1 to ANT
Connections:
- net AIN0: now also U1.4; no longer U2.4
- net DCC: now also U1.47; no longer U2.47
- net DEC2: now also U1.32; no longer U2.32
- net GND: now also U1.31, U1.45, U2.3, U2.P$1; no longer U1.3, U1.P$1, U2.31, U2.45
- net IMU_INT: now also U1.23; no longer U2.23
- net IOA0: now also U1.40; no longer U2.40
- net IOA1: now also U1.41; no longer U2.41
- net IOA2: now also U1.42; no longer U2.42
- net IOA3: now also U1.43; no longer U2.43
- net LED1: now also U1.18; no longer U2.18
- net LED2: now also U1.17; no longer U2.17
- net N$13: now also U1.2; no longer U2.2
- net N$21: now also U1.3; no longer U2.3
- net N$22: now also U1.46; no longer U2.46
- net N$26: now also U1.1; no longer U2.1
- net N$28: now also U1.33; no longer U2.33
- net N$30: now also U1.34; no longer U2.34
- net N$31: now also U1.35; no longer U2.35
- net N$32: now also U1.30; no longer U2.30
- net RESET: now also U1.24; no longer U2.24
- net RX: now also U1.27; no longer U2.27
- net SCL: now also U1.39; no longer U2.39
- net SDA: now also U1.38; no longer U2.38
- net SWDCK: now also U1.25; no longer U2.25
- net SWDIO: now also U1.26; no longer U2.26
- net TX: now also U1.28; no longer U2.28
- net VCC: now also U1.13, U1.36, U1.48, U2.6; no longer U1.6, U2.13, U2.36, U2.48
- net VCCM: now also U2.1; no longer U1.1
Routing:
- net GND: vias 71 -> 72
Other:
- board text added: "+"
- board text added: "ANT"
