File: hardware/dennisquad.sch (EAGLE design)
At the start: 47 parts, among them CN2 HEADER-3X2-PTH, U1 MPU-9250, U10 DRV8839, U2 NRF52832_QFN48, U3 DRV8839, U4 LPS25HB, U5 MCP1700T-3302E/MAY, X1 8Y-32.000MAAV-T, X2 CRYSTAL.ABS07

Commit message: Version 0.9
Parts:
- removed ANT: ANTENNA-BLE, NordicSemi:ANTENNA-BLE
- removed C23, C25: 2.2uF, SparkFun-Capacitors:CAP0402-CAP
- removed C24: 0.47uF, SparkFun-Capacitors:CAP0402-CAP
- removed CN3: (no value), adafruit:JST_2PIN-THM
- removed U$2: FIDUCIAL, jaw:FIDUCIAL
- removed U10: DRV8839, jseng:DRV8839
- removed X2: CRYSTAL.ABS07, abracon:CRYSTAL.ABS07
- added C1: 1.0uF, SparkFun-Capacitors:CAP0603-CAP
- added C2: 4.7pF, SparkFun-Capacitors:CAP0603-CAP
- added JP1: (no value), SparkFun-Connectors:M04X2
- added Q1: FA-128, crystal:FA-128
- added R4: 4k7, SparkFun-Resistors:RESISTOR0402
- added U6: LPS25HB, jaw:LPS25HB
- C10: value 10nF -> 8pF; MPN (none) -> GRM1555C1H8R0BA01D
- C11: value 0.8pf -> 0.8pF; MPN (none) -> GRM1555C2AR80BA01D
- C12: value 8pF -> 2.2uF; MPN (none) -> GRT155R61C225KE13D
- C13: value 100pf -> 0.1uF; MPN (none) -> CL05B104JO5NNNC
- C14, C16: value 12pf -> 0.1uF; MPN (none) -> CL05B104JO5NNNC
- C15: MPN (none) -> CL05B104JO5NNNC
- C17: value 100nf -> 0.1uF; MPN (none) -> CL05B104JO5NNNC
- C18: value 0.1uF -> 10000pF; MPN (none) -> CL05B103KP5NNNC
- C19: value 8pF -> 10uF; device SparkFun-Capacitors:CAP0402-CAP -> SparkFun-Capacitors:CAP0603-CAP; MPN (none) -> C1206C106M4RACAUTO
- C20: value 1.2pf -> 10uF; device SparkFun-Capacitors:CAP0402-CAP -> SparkFun-Capacitors:CAP0603-CAP; MPN (none) -> C1206C106M4RACAUTO
- C21, C5: value .1u -> 0.1uF; MPN (none) -> CL05B104JO5NNNC
- C22, C4: value 10uF -> 0.1uF; device SparkFun-Capacitors:CAP0603-CAP -> SparkFun-Capacitors:CAP0402-CAP; MPN C1206C106M4RACAUTO -> CL05B104JO5NNNC
- C3: value .1u -> 16pF; MPN (none) -> GRM1555C1H160GA01D
- C6: value .1u -> 2.2uF; MPN (none) -> GRT155R61C225KE13D
- C7: value 100nf -> 8pF; MPN (none) -> GRM1555C1H8R0BA01D
- C8: value 100nf -> 16pF; MPN (none) -> GRM1555C1H160GA01D
- C9: value 4.7pf -> 100pF; MPN (none) -> GRM1555C1H101JA01D
- CN1: device jaw:HEADER-2X4 -> adafruit:JST_2PIN-THM
- CN2: value HEADER-3X2-PTH -> (none); device jaw:HEADER-3X2-PTH -> jaw:HEADER-2X4
- L1: MPN (none) -> AISC-0402-3N9J-T
- LED1: MPN (none) -> APHBM2012QBDSURKC
- R3, R6: MPN (none) -> ERJ-2GEJ102X
- R5: MPN (none) -> ERJ-PA2F4701X
- R7: value 4k7 -> 1k; MPN (none) -> ERJ-2GEJ102X
- U$1: value ROBOTMAN-LOGO -> ANTENNA-W3008C; device jaw:ROBOTMAN-LOGO -> SparkFun-RF:ANTENNA-W3008C
- U1: value MPU-9250 -> MCP1700T-3302E/MAY; device template:MPU-9250 -> wrea:MCP1700T-3302E/MAY; MPN (none) -> MCP1700T-3302E/MAY
- U4: value LPS25HB -> DRV8839; device jaw:LPS25HB -> jseng:DRV8839
- U5: value MCP1700T-3302E/MAY -> MPU-9250; device wrea:MCP1700T-3302E/MAY -> template:MPU-9250
- X1: value 8Y-32.000MAAV-T -> CRYSTAL.ABS07; device crystals:TXC-8Y -> abracon:CRYSTAL.ABS07; MPN (none) -> ABS07-120-32.768KHZ-T
- renumbered R8 to R5
Connections:
- removed net AD0/SDO: U1.AD0/SDO
- removed net BOOT0: CN2.P$5
- removed net INT: U1.INT
- new net IMU_INT: U2.P0.20, U5.INT
- new net N$22: C1.1, U2.DEC4
- new net SWDCK: JP1.8, U2.SWDCK
- new net SWDIO: JP1.7, U2.SWDIO
- net AIN0: now also C14.1, R4.1; no longer C5.1, R7.1
- net GND: now also C1.2, C12.1, C16.2, C17.1, C18.2, C2.1, C20.2, C4.1, C9.2, CN1.1, CN2.P$3, CN2.P$6, CN2.P$7, JP1.2, Q1.2, Q1.4, U$1.P$1, U$1.P$2, U4.GND1, U4.GND2, U4.GND_PPAD, U5.AUX_CL, U5.AUX_DA, U5.FSYNC, U5.NCS, U5.RESV@1, U5.RESV@2, U6.GND, U6.SA0; no longer C12.2, C16.1, C17.2, C18.1, C20.1, C23.2, C24.1, C25.1, C4.2, C9.1, CN1.P$2, CN1.P$3, CN1.P$6, CN1.P$7, CN3.1, U1.AUX_CL, U1.AUX_DA, U1.FSYNC, U1.NCS, U1.RESV@2, U10.GND1, U10.GND2, U10.GND_PPAD, U4.GND, U4.SA0, X1.GND
- net IOA2: now also U4.IN1; no longer U10.IN1
- net IOA3: now also U4.IN2; no longer U10.IN2
- net LED1: now also R6.2; no longer R3.2
- net LED2: now also R7.2; no longer R6.2
- net N$12: now also U5.REGOUT; no longer U1.REGOUT
- net N$13: now also C7.1, X1.1; no longer C12.1, X2.1
- net N$14: now also R6.1; no longer R3.1
- net N$15: now also R7.1; no longer R6.1
- net N$16: now also CN2.P$1; no longer CN1.P$1
- net N$17: now also CN2.P$4; no longer CN1.P$4
- net N$18: now also U$1.SIGNAL; no longer ANT.FP, C20.2
- net N$19: now also CN2.P$5, U4.OUT1; no longer CN1.P$5, U10.OUT1
- net N$20: now also CN2.P$8, U4.OUT2; no longer CN1.P$8, U10.OUT2
- net N$21: now also C10.1, X1.2; no longer C19.1, X2.2
- net N$26: now also C5.1; no longer C7.1
- net N$28: now also C9.1; no longer C13.1
- net N$30: now also C8.2, Q1.1; no longer C16.2, X1.1
- net N$31: now also C3.1, Q1.3; no longer C14.1, X1.2
- net RESET: now also JP1.5, R3.1; no longer CN2.P$6
- net RX: now also JP1.6, U2.P0.22; no longer CN2.P$3, U2.P0.11
- net SCL: now also U5.SCL/SCLK, U6.SCL; no longer U1.SCL/SCLK, U4.SCL
- net SDA: now also U5.SDA/SDI, U6.SDA; no longer U1.SDA/SDI, U4.SDA
- net TX: now also JP1.4, U2.P0.23; no longer CN2.P$4, U2.P0.09
- net VCC: now also C12.2, C13.1, C16.1, C17.2, C18.1, C2.2, C22.1, C4.2, JP1.1, R3.2, U1.VOUT, U4.EN1, U4.EN2, U4.NSLEEP, U5.AD0/SDO, U5.RESV, U5.VDD, U5.VDDIO, U6.CS, U6.VCC, U6.VCCIO; no longer C10.1, C17.1, C18.2, C25.2, C3.1, C6.1, C8.2, C9.2, U1.RESV, U1.VDD, U1.VDDIO, U10.EN1, U10.EN2, U10.NSLEEP, U10.VCC, U4.CS, U4.VCCIO, U5.VOUT
- net VCCM: now also C19.1, C20.1, C6.1, CN1.2, R4.2, U1.VIN, U4.VM1, U4.VM2; no longer C22.1, C23.1, C24.2, C4.1, CN2.P$1, CN3.2, R7.2, U10.VM1, U10.VM2, U5.VIN
Other:
- moved on the sheet: C10, C11, C12, C13, C14, C16, C17, C18, C19, C20, C21, C22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

Commit message: Minor fixes
Parts:
- U1: value MCP1700T-3302E/MAY -> NRF52832_QFN48; device wrea:MCP1700T-3302E/MAY -> nRF52Series:NRF52832_QFN48; MPN MCP1700T-3302E/MAY -> (none)
- U2: value NRF52832_QFN48 -> MCP1700T-3302E/MAY; device nRF52Series:NRF52832_QFN48 -> wrea:MCP1700T-3302E/MAY; MPN (none) -> MCP1700T-3302E/MAY
- renumbered U$1 to ANT
Connections:
- net AIN0: now also U1.P0.02/AIN0; no longer U2.P0.02/AIN0
- net GND: now also U1.VSS, U1.VSS2, U2.GND; no longer U1.GND, U2.VSS, U2.VSS2
- net IMU_INT: now also U1.P0.20; no longer U2.P0.20
- net IOA0: now also U1.P0.28/AIN4; no longer U2.P0.28/AIN4
- net IOA1: now also U1.P0.29/AIN5; no longer U2.P0.29/AIN5
- net IOA2: now also U1.P0.30/AIN6; no longer U2.P0.30/AIN6
- net IOA3: now also U1.P0.31/AIN7; no longer U2.P0.31/AIN7
- net LED1: now also U1.P0.15; no longer U2.P0.15
- net LED2: now also U1.P0.14; no longer U2.P0.14
- net N$13: now also U1.P0.00/XL1; no longer U2.P0.00/XL1
- net N$21: now also U1.P0.01/XL2; no longer U2.P0.01/XL2
- net N$22: now also U1.DEC4; no longer U2.DEC4
- net N$26: now also U1.DEC1; no longer U2.DEC1
- net N$28: now also U1.DEC3; no longer U2.DEC3
- net N$30: now also U1.XC1; no longer U2.XC1
- net N$31: now also U1.XC2; no longer U2.XC2
- net N$32: now also U1.ANT; no longer U2.ANT
- net RESET: now also U1.P0.21/RESET; no longer U2.P0.21/RESET
- net RX: now also U1.P0.22; no longer U2.P0.22
- net SCL: now also U1.P0.27; no longer U2.P0.27
- net SDA: now also U1.P0.26; no longer U2.P0.26
- net SWDCK: now also U1.SWDCK; no longer U2.SWDCK
- net SWDIO: now also U1.SWDIO; no longer U2.SWDIO
- net TX: now also U1.P0.23; no longer U2.P0.23
- net VCC: now also U1.VDD, U1.VDD2, U1.VDD3, U2.VOUT; no longer U1.VOUT, U2.VDD, U2.VDD2, U2.VDD3
- net VCCM: now also U2.VIN; no longer U1.VIN
